File: V2A_2.0/V2A_2.0.kicad_pcb (KiCad board)
At the start: 6 copper layers, 94.1 x 135.8 mm, 6 parts, among them J1 1888174-6, J2 1888174-6, J3 1888174-6, J4 1888174-6, J5 IPL1-104-01-L-D-K, J6 IPL1-104-01-L-D-K

Commit message: Needs to breathe
Other:
- outline, holes or cut-outs redrawn
- board text added: "A1"
- board text added: "ASIC PULSE Ground"
- board text added: "B1"
- board text added: "BREATHER HOLE"
- board text added: "DATA / HIGHSPEED"
- board text added: "VD1"
- board text added: "VD2"
- board text removed: "ASIC PULSE - Ground"
